Commit message: 可以稳定使用的版本

File: src/unitree_guide/unitree_ros/robots/a1_description/xacro/gazebo.xacro (robot description, xacro)
@@ -40,11 +40,11 @@
         <sensor name="imu_sensor" type="imu">
             <always_on>true</always_on>
-            <update_rate>400</update_rate>
-            <visualize>true</visualize>
+            <update_rate>200</update_rate>
+            <visualize>false</visualize>
             <topic>__default_topic__</topic>
             <plugin filename="libgazebo_ros_imu_sensor.so" name="imu_plugin">
                 <topicName>trunk_imu</topicName>
                 <bodyName>imu_link</bodyName>
-                <updateRateHZ>400.0</updateRateHZ>
+                <updateRateHZ>200.0</updateRateHZ>
                 <gaussianNoise>0.0</gaussianNoise>
                 <xyzOffset>0 0 0</xyzOffset>
@@ -59,5 +59,5 @@
             <plugin name="${plugin_name}" filename="libgazebo_ros_p3d.so">
                 <alwaysOn>true</alwaysOn>
-                <update_rate>100</update_rate>
+                <update_rate>50</update_rate>
                 <bodyName>${body_name}</bodyName>
                 <topicName>${topic_name}</topicName>
@@ -175,5 +175,5 @@
         <mu1>0.2</mu1>
         <mu2>0.2</mu2>
-        <self_collide>1</self_collide>
+        <self_collide>0</self_collide>
         <material>Gazebo/DarkGrey</material>
         <kp  value="1000000.0"/>
@@ -183,10 +183,10 @@
         <mu1>0.2</mu1>
         <mu2>0.2</mu2>
-        <self_collide>1</self_collide>
+        <self_collide>0</self_collide>
     </gazebo>
     <gazebo reference="FL_foot">
         <mu1>0.6</mu1>
         <mu2>0.6</mu2>
-        <self_collide>1</self_collide>
+        <self_collide>0</self_collide>
         <material>Gazebo/DarkGrey</material>
         <kp  value="1000000.0"/>
@@ -202,5 +202,5 @@
         <mu1>0.2</mu1>
         <mu2>0.2</mu2>
-        <self_collide>1</self_collide>
+        <self_collide>0</self_collide>
         <material>Gazebo/DarkGrey</material>
         <kp  value="1000000.0"/>
@@ -210,10 +210,10 @@
         <mu1>0.2</mu1>
         <mu2>0.2</mu2>
-        <self_collide>1</self_collide>
+        <self_collide>0</self_collide>
     </gazebo>
     <gazebo reference="FR_foot">
         <mu1>0.6</mu1>
         <mu2>0.6</mu2>
-        <self_collide>1</self_collide>
+        <self_collide>0</self_collide>
         <material>Gazebo/DarkGrey</material>
         <kp  value="1000000.0"/>
@@ -229,5 +229,5 @@
         <mu1>0.2</mu1>
         <mu2>0.2</mu2>
-        <self_collide>1</self_collide>
+        <self_collide>0</self_collide>
         <material>Gazebo/DarkGrey</material>
         <kp  value="1000000.0"/>
@@ -237,10 +237,10 @@
         <mu1>0.2</mu1>
         <mu2>0.2</mu2>
-        <self_collide>1</self_collide>
+        <self_collide>0</self_collide>
     </gazebo>
     <gazebo reference="RL_foot">
         <mu1>0.6</mu1>
         <mu2>0.6</mu2>
-        <self_collide>1</self_collide>
+        <self_collide>0</self_collide>
         <material>Gazebo/DarkGrey</material>
         <kp  value="1000000.0"/>
@@ -256,5 +256,5 @@
         <mu1>0.2</mu1>
         <mu2>0.2</mu2>
-        <self_collide>1</self_collide>
+        <self_collide>0</self_collide>
         <material>Gazebo/DarkGrey</material>
         <kp  value="1000000.0"/>
@@ -264,10 +264,10 @@
         <mu1>0.2</mu1>
         <mu2>0.2</mu2>
-        <self_collide>1</self_collide>
+        <self_collide>0</self_collide>
     </gazebo>
     <gazebo reference="RR_foot">
         <mu1>0.6</mu1>
         <mu2>0.6</mu2>
-        <self_collide>1</self_collide>
+        <self_collide>0</self_collide>
         <material>Gazebo/DarkGrey</material>
         <kp  value="1000000.0"/>
@@ -352,11 +352,11 @@
             <sensor name="imu_sensor" type="imu">
                 <always_on>true</always_on>
-                <update_rate>400</update_rate>
-                <visualize>true</visualize>
+                <update_rate>200</update_rate>
+                <visualize>false</visualize>
                 <topic>__default_topic__</topic>
                 <plugin filename="libgazebo_ros_imu_sensor.so" name="imu_plugin">
                     <topicName>/livox/imu</topicName>
                     <bodyName>livox_imu_link</bodyName>
-                    <updateRateHZ>400.0</updateRateHZ>
+                    <updateRateHZ>200.0</updateRateHZ>
                     <gaussianNoise>0.0</gaussianNoise>
                     <xyzOffset>0 0 0</xyzOffset>
@@ -373,11 +373,11 @@
             <sensor type="depth" name="real_sense">
                 <always_on>true</always_on>
-                <update_rate>20.0</update_rate>
+                <update_rate>10.0</update_rate>
                 <camera>
                     <horizontal_fov>${60.0*3.14/180.0}</horizontal_fov>
                     <image>
                         <format>R8G8B8</format>
-                        <width>640</width>
-                        <height>480</height>
+                        <width>320</width>
+                        <height>240</height>
                     </image>
                     <clip>

File: src/unitree_guide/unitree_ros/robots/a1_description/xacro/robot.xacro (robot description, xacro)
@@ -123,5 +123,5 @@
                 <origin xyz="0 0 0" rpy="0 0 0"/>
                 <geometry>
-                    <mesh filename="package://a1_description/meshes/livox_mid360.dae"/>
+                    <box size="0.1 0.1 0.04"/>
                 </geometry>
             </collision>
@@ -188,5 +188,5 @@
                 <origin xyz="0 0 0" rpy="0 0 0"/>
                 <geometry>
-                    <mesh filename="package://a1_description/meshes/d415.stl"/>
+                    <box size="0.099 0.042 0.025"/>
                 </geometry>
             </collision>
