Commit message: 提高激光雷达才杨树，矮小障碍物能检测

File: src/Mid360_imu_sim/urdf/livox_mid360.xacro (robot description, xacro)
@@ -5,5 +5,5 @@
   <xacro:property name="laser_max_range" value="200.0"/>
   <xacro:property name="ros_topic" value="scan"/>
-  <xacro:property name="samples" value="24000"/>
+  <xacro:property name="samples" value="48000"/>
   <xacro:property name="downsample" value="1"/>
   <xacro:macro name="null_inertial">
